File: hardware/effective-pancake-HMI/effective-pancake-HMI.sch (KiCad schematic (older format))
At the start: 37 parts, among them SW1 SW_SPST, SW2 SW_SPST, SW3 SW_SPST, SW4 SW_SPST, U1 ATmega328P-PU, U2 R-78C5.0-1.0, Y1 Crystal

Commit message: Finished schematics, fp association, and verifications.
Parts:
- removed C_POR1: C_Small, symbol Device:C_Small
- C_AVR1, C_AVR2: value 10nF -> 100nF; footprint (none) -> Capacitor_SMD:C_0805_2012Metric_Pad1.15x1.40mm_HandSolder
- C_osc1, C_osc2: value C_Small -> 22pF; footprint (none) -> Capacitor_SMD:C_1206_3216Metric_Pad1.42x1.75mm_HandSolder
- D1, D2, D3, D_pwr1: footprint (none) -> LED_THT:LED_D5.0mm_Clear
- D_pp1: value D_Zener_Small -> BZX84 - 12V; footprint (none) -> Diode_SMD:D_SOT-23_ANK
- J_EXT_UART1: footprint (none) -> Connector_PinHeader_2.54mm:PinHeader_1x06_P2.54mm_Vertical
- J_I2C1: footprint (none) -> Connector_JST:JST_XH_B4B-XH-A_1x04_P2.50mm_Vertical
- J_ICSP1: footprint (none) -> Connector_IDC:IDC-Header_2x03_P2.54mm_Vertical
- J_IDC_EXT1: footprint (none) -> Connector_IDC:IDC-Header_2x04_P2.54mm_Vertical
- KEY1, KEY2, SW_RST1: footprint (none) -> digikey-footprints:Switch_Tactile_SMD_6x6mm
- Q_pp1: footprint (none) -> Package_TO_SOT_SMD:SOT-23
- RE1: footprint (none) -> Rotary_Encoder:RotaryEncoder_Alps_EC12E_Vertical_H20mm
- R_A1, R_B1: value 2.7K -> 10K; footprint (none) -> Resistor_SMD:R_0805_2012Metric_Pad1.15x1.40mm_HandSolder
- R_LED1, R_LED2, R_LED3: value R_Small -> 1K; footprint (none) -> Resistor_SMD:R_0805_2012Metric_Pad1.15x1.40mm_HandSolder
- R_SCL1, R_SDA1: footprint (none) -> Resistor_SMD:R_0805_2012Metric_Pad1.15x1.40mm_HandSolder
- R_osc1: footprint (none) -> Resistor_SMD:R_1206_3216Metric_Pad1.42x1.75mm_HandSolder
- R_pwr1: value R_Small -> 5.1K; footprint (none) -> Resistor_SMD:R_0805_2012Metric_Pad1.15x1.40mm_HandSolder
- R_rpp1: value R_Small -> 15k; footprint (none) -> Resistor_SMD:R_0805_2012Metric_Pad1.15x1.40mm_HandSolder
- R_rst1: renamed from R_POR1; footprint (none) -> Resistor_SMD:R_0805_2012Metric_Pad1.15x1.40mm_HandSolder
- SW1, SW2, SW3, SW4: value SW_SPST -> EG5617-ND; footprint (none) -> effective-pancake-HMI:Rocker Switch RA11131121
- Y_osc1: renamed from Y1; value Crystal -> 16MHz; footprint (none) -> Crystal:Crystal_SMD_HC49-SD
Other:
- moved on the sheet: R_rst1
